File: rumblesan-template/rumblesan-template.kicad_pcb (KiCad board)
At the start: 2 copper layers, 0 parts

Commit message: Tweaks to template
Other:
- rule pad_to_mask_clearance: 0.0508 -> 0
Changed lines of the file:
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@@
     (pad_size 1.524 1.524)
     (pad_drill 0.762)
-    (pad_to_mask_clearance 0.0508)
-    (solder_mask_min_width 0.127)
+    (pad_to_mask_clearance 0)
     (aux_axis_origin 0 0)
     (visible_elements FFFFFF7F)
     (pcbplotparams
-      (layerselection 0x010fc_ffffffff)
-      (usegerberextensions false)
+      (layerselection 0x010f0_ffffffff)
+      (usegerberextensions true)
       (usegerberattributes true)
       (usegerberadvancedattributes true)
@@
       (psa4output false)
       (plotreference true)
-      (plotvalue true)
+      (plotvalue false)
       (plotinvisibletext false)
       (padsonsilk false)
@@
       (outputformat 1)
       (mirror false)
-      (drillshape 1)
+      (drillshape 0)
       (scaleselection 1)
       (outputdirectory ""))

Commit message: Updating template
Other:
- net class Default removed
- net class Power removed
- net class Signal removed
Changed lines of the file:
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@@
-(kicad_pcb (version 20171130) (host pcbnew "(5.1.8-0-10_14)")
+(kicad_pcb (version 20211014) (generator pcbnew)
   (general
     (thickness 1.6)
-    (drawings 0)
-    (tracks 0)
-    (zones 0)
-    (modules 0)
-    (nets 1)
   )
-  (page A4)
+  (paper "A4")
+  (title_block
+    (comment 2 "creativecommons.org/licenses/by/4.0")
+    (comment 3 "License: CC BY 4.0")
+    (comment 4 "Author: Guy John")
+  )
   (layers
-    (0 F.Cu signal)
-    (31 B.Cu signal)
-    (36 B.SilkS user)
-    (37 F.SilkS user)
-    (38 B.Mask user)
-    (39 F.Mask user)
-    (41 Cmts.User user)
-    (44 Edge.Cuts user)
-    (45 Margin user)
-    (46 B.CrtYd user)
-    (47 F.CrtYd user)
-    (48 B.Fab user)
-    (49 F.Fab user)
+    (0 "F.Cu" signal)
+    (31 "B.Cu" signal)
+    (36 "B.SilkS" user "B.Silkscreen")
+    (37 "F.SilkS" user "F.Silkscreen")
+    (38 "B.Mask" user)
+    (39 "F.Mask" user)
+    (41 "Cmts.User" user "User.Comments")
+    (44 "Edge.Cuts" user)
+    (45 "Margin" user)
+    (46 "B.CrtYd" user "B.Courtyard")
+    (47 "F.CrtYd" user "F.Courtyard")
+    (48 "B.Fab" user)
+    (49 "F.Fab" user)
   )
   (setup
-    (last_trace_width 0.254)
-    (user_trace_width 0.2032)
-    (user_trace_width 0.3048)
-    (user_trace_width 0.635)
-    (user_trace_width 1.27)
-    (trace_clearance 0.254)
-    (zone_clearance 0.508)
-    (zone_45_only no)
-    (trace_min 0.2032)
-    (via_size 0.762)
-    (via_drill 0.381)
-    (via_min_size 0.4064)
-    (via_min_drill 0.3048)
-    (uvia_size 0.762)
-    (uvia_drill 0.381)
-    (uvias_allowed no)
-    (uvia_min_size 0.2032)
-    (uvia_min_drill 0.1016)
-    (edge_width 0.05)
-    (segment_width 0.2)
-    (pcb_text_width 0.3)
-    (pcb_text_size 1.5 1.5)
-    (mod_edge_width 0.12)
-    (mod_text_size 1 1)
-    (mod_text_width 0.15)
-    (pad_size 1.524 1.524)
-    (pad_drill 0.762)
     (pad_to_mask_clearance 0)
-    (aux_axis_origin 0 0)
-    (visible_elements FFFFFF7F)
     (pcbplotparams
-      (layerselection 0x010f0_ffffffff)
+      (layerselection 0x00010f0_ffffffff)
+      (disableapertmacros false)
       (usegerberextensions true)
       (usegerberattributes true)
       (usegerberadvancedattributes true)
       (creategerberjobfile true)
+      (svguseinch false)
+      (svgprecision 6)
       (excludeedgelayer true)
-      (linewidth 0.100000)
       (plotframeref false)
       (viasonmask false)
@@
       (hpglpenspeed 20)
       (hpglpendiameter 15.000000)
+      (dxfpolygonmode true)
+      (dxfimperialunits true)
+      (dxfusepcbnewfont true)
       (psnegative false)
       (psa4output false)
@@
       (plotvalue false)
       (plotinvisibletext false)
-      (padsonsilk false)
+      (sketchpadsonfab false)
       (subtractmaskfromsilk false)
       (outputformat 1)
@@
       (drillshape 0)
       (scaleselection 1)
-      (outputdirectory ""))
+      (outputdirectory "")
+    )
   )
   (net 0 "")
-  (net_class Default "This is the default net class."
-    (clearance 0.254)
-    (trace_width 0.254)
-    (via_dia 0.762)
-    (via_drill 0.381)
-    (uvia_dia 0.762)
-    (uvia_drill 0.381)
-    (diff_pair_width 0.2032)
-    (diff_pair_gap 0.254)
-  )
-  (net_class Power ""
-    (clearance 0.3048)
-    (trace_width 0.635)
-    (via_dia 0.762)
-    (via_drill 0.381)
-    (uvia_dia 0.762)
-    (uvia_drill 0.381)
-    (diff_pair_width 0.2032)
-    (diff_pair_gap 0.254)
-  )
-  (net_class Signal ""
-    (clearance 0.3048)
-    (trace_width 0.3048)
-    (via_dia 0.762)
-    (via_drill 0.381)
-    (uvia_dia 0.762)
-    (uvia_drill 0.381)
-    (diff_pair_width 0.2032)
-    (diff_pair_gap 0.254)
-  )
 )
